Commit message: Add tuned camera rig + headless sim env with viewer/teleop/cam modes (subtask 1+2)
- cameras.py: side cam tuned interactively (pos + pan/tilt/roll, baked as
  inputs and computed to lookat/up at resolve time); wrist cam offset; base
  anchor fixed to the table top (0.74) instead of the stale floor-level 0.1.
- so101_new_calib.urdf + meshes: add the camera_wrist mount frame that the
  wrist camera attaches to.
- sim_env.py: gym-style SimEnv (reset/step/observation) producing the
  MolmoAct2 observation (top+side+wrist RGB + 6-D state). Modes: headless PNG
  snapshot, --viewer (3D window), --cams (live OpenCV windows), --teleop
  (viewer + keyboard joint control + live camera windows, render throttled
  every 16 steps since 3 cam renders ~7ms dominate the 0.2ms sim step).
- arm_cam_view.py / wrist_cam_tuner.py: the web-UI tuners used to dial the poses.

Co-Authored-By: Claude Opus 4.8 (1M context) <noreply@anthropic.com>

File: assets/so101/so101_new_calib.urdf (robot description, URDF)
Before this commit: robot so101_new_calib, 8 links, 7 joints
Links:
- added link camera_wrist, mass 1e-6
Joints:
- added joint wrist_to_camera_wrist: type fixed, parent gripper_link, child camera_wrist, origin xyz=0.002265 -0.074668 0.009659 rpy=0.437925 0 0
